File: ele/Mickoflus.sch (EAGLE design)
At the start: 63 parts, among them IC1 74HC595D, IC2 74HC595D

Commit message: Jarek's editations of the schematics.
Parts:
- removed JP10: (no value), pinhead:PINHD-1X4
- added JP20: (no value), pinhead:PINHD-1X5
- added JP21: (no value), pinhead:PINHD-1X6
- JP19: device pinhead:PINHD-1X4 -> pinhead:PINHD-1X5
- JP9: device pinhead:PINHD-1X4 -> pinhead:PINHD-1X6
Connections:
- new net N$26: JP21.1
- new net N$41: JP21.6
- net +3V3: now also JP19.4, JP20.4; no longer JP19.3
- net +5V: now also JP19.5, JP20.5, JP21.2, JP9.2; no longer JP10.4, JP5.4, JP9.4
- net ENC1A: now also JP9.3; no longer JP9.1
- net ENC1B: now also JP9.4; no longer JP9.2
- net ENC2A: now also JP21.3; no longer JP10.1
- net ENC2B: now also JP21.4; no longer JP10.2
- net GND: now also JP19.3, JP20.3, JP21.5, JP9.5; no longer JP10.3, JP19.4, JP9.3
- net N$15: now also JP9.6
- net N$2: now also JP9.1
- net SCL: now also JP20.1
- net SDA: now also JP20.2
Other:
- note added: "//todo: PCA expander - 16 pinů - GND, SIG, 3V3 overit input nebo output only piny specialni konektor na chytre LEDky, accelerometer, ...? ochrana proti podvybití baterie stromopinheadiste s GND, 5V (DPS step-down), SIG, SIG, GND, 3V3"
- note removed: "//todo: PCA expander 5V stabilizer overit input nebo output only piny specialni konektor na chytre LEDky, accelerometer, ...?"
- moved on the sheet: D2, IC4, M4-1, M4-2, M8-1, M8-2, R4, R5
